Commit message: mtc_tutorial adapted to dynamic vector and wilson_sim broken

File: src/wilson/ros2_control/wilson_system.ros2_control.xacro (robot description, xacro)
@@ -124,18 +124,13 @@
       </joint>
       <!-- gripper_right_finger_joint is now a mimic joint, no control interfaces needed -->
-      <!--
       <joint name="gripper_right_finger_joint">
         <command_interface name="position">
-          <param name="min">-0</param>
-          <param name="max">0.05</param>
+          <param name="min">-0.05</param>
+          <param name="max">0.0</param>
         </command_interface>
         <state_interface name="position">
           <param name="initial_value">0.0</param>
         </state_interface>
-        <state_interface name="velocity">
-          <param name="initial_value">0.0</param>
-        </state_interface>
       </joint>
-      -->
       <!--
       <joint name="end_effector_roll_joint">

File: src/wilson/urdf/wilson_core.xacro (robot description, xacro)
@@ -619,8 +619,4 @@
       effort="0"
       velocity="0" />
-    <mimic
-      joint="gripper_left_finger_joint"
-      multiplier="-1"
-      offset="0" />
   </joint>
 </robot>

File: src/wilson_moveit_config/config/wilson.ros2_control.xacro (robot description, xacro)
@@ -36,4 +36,18 @@
                 <state_interface name="velocity"/>
             </joint>
+            <joint name="end_effector_roll_joint">
+                <command_interface name="position"/>
+                <state_interface name="position">
+                  <param name="initial_value">${initial_positions['end_effector_roll_joint']}</param>
+                </state_interface>
+                <state_interface name="velocity"/>
+            </joint>
+            <joint name="end_effector_yaw_joint">
+                <command_interface name="position"/>
+                <state_interface name="position">
+                  <param name="initial_value">${initial_positions['end_effector_yaw_joint']}</param>
+                </state_interface>
+                <state_interface name="velocity"/>
+            </joint>
             <joint name="gripper_left_finger_joint">
                 <command_interface name="position"/>
@@ -43,4 +57,11 @@
                 <state_interface name="velocity"/>
             </joint>
+            <joint name="gripper_right_finger_joint">
+                <command_interface name="position"/>
+                <state_interface name="position">
+                  <param name="initial_value">${initial_positions['gripper_right_finger_joint']}</param>
+                </state_interface>
+                <state_interface name="velocity"/>
+            </joint>
         </ros2_control>
     </xacro:macro>

Commit message: wilson arm to target pose working.

File: src/wilson/ros2_control/wilson_system.ros2_control.xacro (robot description, xacro)
@@ -133,5 +133,4 @@
         </state_interface>
       </joint>
-      <!--
       <joint name="end_effector_roll_joint">
         <command_interface name="position">
@@ -140,7 +139,4 @@
         </command_interface>
         <state_interface name="position">
-          <param name="initial_value">0.0</param>
-        </state_interface>
-        <state_interface name="velocity">
           <param name="initial_value">0.0</param>
         </state_interface>
@@ -154,9 +150,5 @@
           <param name="initial_value">0.0</param>
         </state_interface>
-        <state_interface name="velocity">
-          <param name="initial_value">0.0</param>
-        </state_interface>
       </joint>
-      -->
     </ros2_control>
   </xacro:macro>

File: src/wilson/urdf/end_effector.xacro (robot description, xacro)
@@ -4,12 +4,10 @@
     <xacro:property name="green" value="0.2 0.8 0.2 1.0"/>
     <!-- End effector frame (for convenience in motion planning) -->
-    <joint name="end_effector_roll_joint" type="fixed">
+    <joint name="end_effector_roll_joint" type="revolute">
         <parent link="gripper_base"/>
         <child link="end_effector_roll"/>
         <origin xyz="${end_effector_offset_x} 0 0" rpy="0 0 0"/>
-        <!--
         <axis xyz="1 0 0"/>
         <limit effort="0.0" lower="-3.14" upper="3.14" velocity="1"/>
-    -->
     </joint>
     <link name="end_effector_roll">
@@ -24,12 +22,10 @@
         </visual>
     </link>
-    <joint name="end_effector_yaw_joint" type="fixed">
+    <joint name="end_effector_yaw_joint" type="revolute">
         <parent link="end_effector_roll"/>
         <child link="end_effector_yaw"/>
         <origin xyz="0 0 0" rpy="0 0 0"/>
-        <!--
         <axis xyz="0 0 1"/>
         <limit effort="0.0" lower="-3.14" upper="3.14" velocity="1"/>
-    -->
     </joint>
     <link name="end_effector_yaw">
