Commit message: Locate drink displays image and camera topics fixed

File: src/wilson/urdf/camera.xacro (robot description, xacro)
@@ -2,15 +2,15 @@
 <robot xmlns:xacro="http://www.ros.org/wiki/xacro" >
     <joint name="camera_optical_joint" type="fixed">
-        <parent link="camera_link"/>
+        <parent link="camera_sensor_link"/>
         <child link="camera_link_optical"/>
         <origin xyz="0 0 0" rpy="${-pi/2} 0 ${-pi/2}"/>
     </joint>
     <link name="camera_link_optical"></link>
-    <gazebo reference="camera_link">
+    <gazebo reference="camera_sensor_link">
         <material>Gazebo/Black</material>
-        <sensor name="camera" type="camera">
+        <sensor name="rgb_camera" type="camera">
             <pose> 0 0 0 0 0 0 </pose>
             <visualize>true</visualize>
-            <update_rate>5</update_rate>
+            <update_rate>20</update_rate>
             <camera>
                 <horizontal_fov>1.089</horizontal_fov>
@@ -21,5 +21,5 @@
                 </image>
                 <clip>
-                    <near>0.05</near>
+                    <near>0.4</near>
                     <far>8.0</far>
                 </clip>

File: src/wilson/urdf/depth_camera.xacro (robot description, xacro)
@@ -2,15 +2,15 @@
 <robot xmlns:xacro="http://www.ros.org/wiki/xacro" >
     <joint name="depth_camera_optical_joint" type="fixed">
-        <parent link="depth_camera_link"/>
+        <parent link="depth_camera_sensor_link"/>
         <child link="depth_camera_link_optical"/>
         <origin xyz="0 0 0" rpy="${-pi/2} 0 ${-pi/2}"/>
     </joint>
     <link name="depth_camera_link_optical"></link>
-    <gazebo reference="depth_camera_link">
+    <gazebo reference="depth_camera_sensor_link">
         <material>Gazebo/Black</material>
-        <sensor name="camera" type="depth">
+        <sensor name="depth_camera" type="depth">
             <pose> 0 0 0 0 0 0 </pose>
             <visualize>true</visualize>
-            <update_rate>5</update_rate>
+            <update_rate>20</update_rate>
             <camera>
                 <horizontal_fov>1.089</horizontal_fov>
@@ -21,12 +21,12 @@
                 </image>
                 <clip>
-                    <near>0.05</near>
-                    <far>8.0</far>
+                    <near>0.5</near>
+                    <far>4.0</far>
                 </clip>
             </camera>
             <plugin name="depth_camera_controller" filename="libgazebo_ros_camera.so">
                 <frame_name>depth_camera_link_optical</frame_name>
-                <mindepth>0.1</mindepth>
-                <maxdepth>100.0</maxdepth>
+                <mindepth>0.5</mindepth>
+                <maxdepth>4.0</maxdepth>
             </plugin>
         </sensor>

File: src/wilson/urdf/wilson_core.xacro (robot description, xacro)
@@ -166,4 +166,21 @@
       xyz="0 0 0" />
   </joint>
+  <!-- Sensor origin link offset 45cm behind the camera housing to work around Open3D's 0.5m minimum clip distance -->
+  <link
+    name="camera_sensor_link">
+  </link>
+  <joint
+    name="camera_sensor_joint"
+    type="fixed">
+    <origin
+      xyz="-0.25 0 0"
+      rpy="0 0 0" />
+    <parent
+      link="camera_link" />
+    <child
+      link="camera_sensor_link" />
+    <axis
+      xyz="0 0 0" />
+  </joint>
   <link
     name="depth_camera_link">
@@ -219,4 +236,21 @@
       xyz="0 0 0" />
   </joint>
+  <!-- Sensor origin link offset 25cm behind the camera housing to work around Open3D's 0.5m minimum clip distance -->
+  <link
+    name="depth_camera_sensor_link">
+  </link>
+  <joint
+    name="depth_camera_sensor_joint"
+    type="fixed">
+    <origin
+      xyz="-0.25 0 0"
+      rpy="0 0 0" />
+    <parent
+      link="depth_camera_link" />
+    <child
+      link="depth_camera_sensor_link" />
+    <axis
+      xyz="0 0 0" />
+  </joint>
   <link
     name="link_1">
